File: buck_converter.kicad_sch (KiCad schematic)
At the start: 17 parts, among them J1 Screw_Terminal_01x02, J2 Screw_Terminal_01x02

Commit message: Fixed
Parts:
- removed C1A1, C2A1, C2B1: 22uF, Capacitor_THT:CP_Radial_D6.3mm_P2.50mm, symbol Device:C
- removed C1B1: 0.1uF, Capacitor_THT:C_Disc_D5.0mm_W2.5mm_P5.00mm, symbol Device:C
- removed R6: 10k, Resistor_THT:R_Axial_DIN0207_L6.3mm_D2.5mm_P7.62mm_Horizontal, symbol Device:R
- removed U1: ~, Package_TO_SOT_SMD:SOT-583-8, symbol New_Library:MP2338
- added C1, C2, C6: 22u, Capacitor_SMD:C_1206_3216Metric_Pad1.33x1.80mm_HandSolder, symbol Device:C
- added Q1: SUD09P10-195, Package_TO_SOT_SMD:TO-252-2, symbol Transistor_FET:SUD09P10-195
- added RV1: 20K, Potentiometer_THT:Potentiometer_Bourns_3296W_Vertical, symbol Device:R_Potentiometer
- added U1: TPS54308, Package_TO_SOT_SMD:SOT-23-6, symbol Regulator_Switching:TPS54308
- C3: value 0.1uF -> 100n; footprint Capacitor_THT:C_Disc_D5.0mm_W2.5mm_P5.00mm -> Capacitor_SMD:C_0805_2012Metric_Pad1.18x1.45mm_HandSolder
- C4: value 22nF -> 100n; footprint Capacitor_THT:C_Disc_D5.0mm_W2.5mm_P5.00mm -> Capacitor_SMD:C_0805_2012Metric_Pad1.18x1.45mm_HandSolder
- C5: value 300pF -> 22u; footprint Capacitor_THT:C_Disc_D5.0mm_W2.5mm_P5.00mm -> Capacitor_SMD:C_1206_3216Metric_Pad1.33x1.80mm_HandSolder
- J1: value Screw_Terminal_01x02 -> Input Screw Terminal; footprint TerminalBlock_Phoenix:TerminalBlock_Phoenix_MKDS-1,5-2-5.08_1x02_P5.08mm_Horizontal -> Connector_Phoenix_MC_HighVoltage:PhoenixContact_MC_1,5_2-G-5.08_1x02_P5.08mm_Horizontal
- J2: value Screw_Terminal_01x02 -> Output Screw Terminal; footprint TerminalBlock_Phoenix:TerminalBlock_Phoenix_MKDS-1,5-2-5.08_1x02_P5.08mm_Horizontal -> Connector_Phoenix_MC_HighVoltage:PhoenixContact_MC_1,5_2-G-5.08_1x02_P5.08mm_Horizontal
- L1: value 6.6uH -> 15u; footprint Inductor_THT:L_Radial_D10.0mm_P5.00mm_Neosid_SD12k_style3 -> Inductor_SMD:L_Bourns_SRP1038C_10.0x10.0mm
- R1: value 90.9k -> 100K; footprint Resistor_THT:R_Axial_DIN0207_L6.3mm_D2.5mm_P7.62mm_Horizontal -> Resistor_SMD:R_0805_2012Metric_Pad1.20x1.40mm_HandSolder
- R2: value 10k -> 100K; footprint Resistor_THT:R_Axial_DIN0207_L6.3mm_D2.5mm_P7.62mm_Horizontal -> Resistor_SMD:R_0805_2012Metric_Pad1.20x1.40mm_HandSolder
- R3: value 191k -> 100K; footprint Resistor_THT:R_Axial_DIN0207_L6.3mm_D2.5mm_P7.62mm_Horizontal -> Resistor_SMD:R_0805_2012Metric_Pad1.20x1.40mm_HandSolder
- R4: value 49.9k -> 100K; footprint Resistor_THT:R_Axial_DIN0207_L6.3mm_D2.5mm_P7.62mm_Horizontal -> Resistor_SMD:R_0805_2012Metric_Pad1.20x1.40mm_HandSolder
- R5: value 10k -> 5K; footprint Resistor_THT:R_Axial_DIN0207_L6.3mm_D2.5mm_P7.62mm_Horizontal -> Resistor_SMD:R_0805_2012Metric_Pad1.20x1.40mm_HandSolder
Connections:
- net GND: now also C3.2, C5.2, J1.1 (Pin_1), J2.1 (Pin_1), R3.2, C1.2, C2.2, C6.2, Q1.1 (G), RV1.3, U1.1 (GND); no longer C4.2, J1.2 (Pin_2), J2.2 (Pin_2), R2.2, R4.2
- net VOUT: now also C5.1, J2.2 (Pin_2), R4.1, C6.1; no longer C5.2, J2.1 (Pin_1), R1.2, R5.2
- net SW: now reaches L1.1
- net SW: now also C4.2, U1.2 (SW); no longer C3.2
- net FB: now reaches R5.1
- net FB: now also R4.2, U1.4 (FB)
- net VIN_P: now reaches C3.1
- net VIN_P: now also R1.1, C2.1, Q1.3 (S), U1.3 (VIN)
- net at C4.1: now also U1.6 (BOOT)
- net 24V renamed EN
- net EN: now also R2.2, U1.5 (EN); no longer J1.1 (Pin_1)
- new net: R5.2, RV1.2
- new net: R1.2, R2.1
- new net VIN: C1.1, J1.2 (Pin_2), Q1.2 (D)
- no-connect marks 0 -> 1
Other:
- note added: "3296W-1-203LF"
- note added: "3A Buck Converter"
- note added: "Input Terminal"
- note added: "Notes - Vin is limited to max gate VGS on the input reverse protection MOSFET and limited by Ven. - Vout can be set changing Vfb using R Trimmer. Formulas - Ven = {R3/(R1+R2) + R3]}Vin *Voltage Divider Formula => (100K / 300K) Vin - Lmin = Vout(Vinmax - Vout) / Vinmaax x Kind x Iout x Fsw *Equation 8 in the datasheet Assuming Iout = 3A, Fsw = 350Khz, Kind = 0.3 , Vinmax = 18V => @Vout = 3.3V => 3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"
- note added: "Output Terminal"
- note added: "SRP1038A-150M"
- title: (none) -> DC-DC 3A Buck Converter
